File: pcb/hdmi-breakout/hdmi-breakout.kicad_pcb (KiCad board)
At the start: 4 copper layers, 35 x 29 mm, 4 parts, among them J1 Conn_01x09, J2 HDMI_A_1.4, J3 HDMI_A_1.4, J4 Conn_01x09

Commit message: correct hardware bugs
Parts:
- added R1: 100k, Resistor_SMD:R_0603_1608Metric_Pad0.98x0.95mm_HandSolder, F.Cu at (120.5, 115.3)
- added R2: 100k, Resistor_SMD:R_0603_1608Metric_Pad0.98x0.95mm_HandSolder, F.Cu at (117.3, 115.3)
Connections:
- J4 pad 4: SCL -> Net-(J4-Pin_4)
- J4 pad 5: SDA -> Net-(J4-Pin_5)
Routing:
- net SDA: track 52.5 -> 42.3 mm
- net Net-(J4-Pin_5): track 0.00 -> 5.10 mm
- net Net-(J4-Pin_4): track 0.00 -> 4.44 mm
- net SCL: track 53.5 -> 54.7 mm

Commit message: update name
Other:
- board text added: "github.com/flaviut/ceclink"
- board text removed: "github.com/gkoh/pico-cec"
Changed lines of the file:
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@@
 		)
 	)
-	(gr_text "github.com/gkoh/pico-cec"
+	(gr_text "github.com/flaviut/ceclink"
 		(at 133.001868 118.00184 0)
 		(layer "B.SilkS")
@@
 	)
 	(segment
+		(start 117.251868 116.16434)
+		(end 117.251868 117.631868)
+		(width 0.254)
+		(layer "F.Cu")
+		(net "Net-(J4-Pin_4)")
+	)
+	(segment
+		(start 117.251868 117.631868)
+		(end 119.350592 119.730592)
+		(width 0.254)
+		(layer "F.Cu")
+		(net "Net-(J4-Pin_4)")
+	)
+	(segment
+		(start 107.91165 101.95094)
+		(end 125.808185 101.95094)
+		(width 0.254)
+		(layer "F.Cu")
+		(net "SCL")
+	)
+	(segment
+		(start 127.501868 109.50184)
+		(end 127.501868 105.314643)
+		(width 0.254)
+		(layer "F.Cu")
+		(net "SCL")
+	)
+	(segment
+		(start 123.116034 116.50184)
+		(end 121.857534 115.24334)
+		(width 0.254)
+		(layer "F.Cu")
+		(net "SCL")
+	)
+	(segment
+		(start 121.857534 115.24334)
+		(end 118.155868 115.24334)
+		(width 0.254)
+		(layer "F.Cu")
+		(net "SCL")
+	)
+	(segment
+		(start 128.001868 116.00184)
+		(end 128.001868 110.00184)
+		(width 0.254)
+		(layer "F.Cu")
+		(net "SCL")
+	)
+	(segment
+		(start 125.808185 101.95094)
+		(end 128.098768 104.241523)
+		(width 0.254)
+		(layer "F.Cu")
+		(net "SCL")
+	)
+	(segment
+		(start 127.838541 105.314643)
+		(end 127.501868 105.314643)
+		(width 0.254)
+		(layer "F.Cu")
+		(net "SCL")
+	)
+	(segment
+		(start 128.098768 105.054416)
+		(end 127.838541 105.314643)
+		(width 0.254)
+		(layer "F.Cu")
+		(net "SCL")
+	)
+	(segment
+		(start 118.155868 115.24334)
+		(end 117.251868 114.33934)
+		(width 0.254)
+		(layer "F.Cu")
+		(net "SCL")
+	)
+	(segment
+		(start 110.2981 105.01)
+		(end 107.55514 105.01)
+		(width 0.254)
+		(layer "F.Cu")
+		(net "SCL")
+	)
+	(segment
+		(start 106.9352 104.39006)
+		(end 106.9352 102.927389)
+		(width 0.254)
+		(layer "F.Cu")
+		(net "SCL")
+	)
+	(segment
+		(start 128.001868 116.00184)
+		(end 127.501868 116.50184)
+		(width 0.254)
+		(layer "F.Cu")
+		(net "SCL")
+	)
+	(segment
+		(start 107.55514 105.01)
+		(end 106.9352 104.39006)
+		(width 0.254)
+		(layer "F.Cu")
+		(net "SCL")
+	)
+	(segment
+		(start 106.9352 102.927389)
+		(end 107.91165 101.95094)
+		(width 0.254)
+		(layer "F.Cu")
+		(net "SCL")
+	)
+	(segment
+		(start 128.001868 110.00184)
+		(end 127.501868 109.50184)
+		(width 0.254)
+		(layer "F.Cu")
+		(net "SCL")
+	)
+	(segment
+		(start 127.501868 116.50184)
+		(end 123.116034 116.50184)
+		(width 0.254)
+		(layer "F.Cu")
+		(net "SCL")
+	)
+	(segment
+		(start 128.098768 104.241523)
+		(end 128.098768 105.054416)
+		(width 0.254)
+		(layer "F.Cu")
+		(net "SCL")
+	)
+	(via
+		(at 127.501868 105.314643)
+		(size 0.6858)
+		(drill 0.3302)
+		(layers "F.Cu" "B.Cu")
+		(net "SCL")
+	)
+	(segment
+		(start 126.3521 105.01)
+		(end 124.7981 105.01)
+		(width 0.254)
+		(layer "B.Cu")
+		(net "SCL")
+	)
+	(segment
+		(start 126.656743 105.314643)
+		(end 126.3521 105.01)
+		(width 0.254)
+		(layer "B.Cu")
+		(net "SCL")
+	)
+	(segment
+		(start 127.501868 105.314643)
+		(end 126.656743 105.314643)
+		(width 0.254)
+		(layer "B.Cu")
+		(net "SCL")
+	)
+	(segment
 		(start 110.2981 112.01)
 		(end 112.248101 112.01)
@@
 	)
 	(segment
-		(start 107.91165 101.95094)
-		(end 125.808185 101.95094)
-		(width 0.254)
-		(layer "F.Cu")
-		(net "SCL")
-	)
-	(segment
-		(start 127.501868 109.50184)
-		(end 127.501868 105.314643)
-		(width 0.254)
-		(layer "F.Cu")
-		(net "SCL")
-	)
-	(segment
-		(start 123.116034 116.50184)
-		(end 121.857534 115.24334)
-		(width 0.254)
-		(layer "F.Cu")
-		(net "SCL")
-	)
-	(segment
-		(start 121.857534 115.24334)
-		(end 118.155868 115.24334)
-		(width 0.254)
-		(layer "F.Cu")
-		(net "SCL")
-	)
-	(segment
-		(start 128.001868 116.00184)
-		(end 128.001868 110.00184)
-		(width 0.254)
-		(layer "F.Cu")
-		(net "SCL")
-	)
-	(segment
-		(start 125.808185 101.95094)
-		(end 128.098768 104.241523)
-		(width 0.254)
-		(layer "F.Cu")
-		(net "SCL")
-	)
-	(segment
-		(start 127.838541 105.314643)
-		(end 127.501868 105.314643)
-		(width 0.254)
-		(layer "F.Cu")
-		(net "SCL")
-	)
-	(segment
-		(start 128.098768 105.054416)
-		(end 127.838541 105.314643)
-		(width 0.254)
-		(layer "F.Cu")
-		(net "SCL")
-	)
-	(segment
-		(start 118.155868 115.24334)
-		(end 117.251868 114.33934)
-		(width 0.254)
-		(layer "F.Cu")
-		(net "SCL")
-	)
-	(segment
-		(start 110.2981 105.01)
-		(end 107.55514 105.01)
-		(width 0.254)
-		(layer "F.Cu")
-		(net "SCL")
-	)
-	(segment
-		(start 106.9352 104.39006)
-		(end 106.9352 102.927389)
-		(width 0.254)
-		(layer "F.Cu")
-		(net "SCL")
-	)
-	(segment
-		(start 128.001868 116.00184)
-		(end 127.501868 116.50184)
-		(width 0.254)
-		(layer "F.Cu")
-		(net "SCL")
-	)
-	(segment
-		(start 107.55514 105.01)
-		(end 106.9352 104.39006)
-		(width 0.254)
-		(layer "F.Cu")
-		(net "SCL")
-	)
-	(segment
-		(start 106.9352 102.927389)
-		(end 107.91165 101.95094)
-		(width 0.254)
-		(layer "F.Cu")
-		(net "SCL")
-	)
-	(segment
-		(start 128.001868 110.00184)
-		(end 127.501868 109.50184)
-		(width 0.254)
-		(layer "F.Cu")
-		(net "SCL")
-	)
-	(segment
-		(start 127.501868 116.50184)
-		(end 123.116034 116.50184)
-		(width 0.254)
-		(layer "F.Cu")
-		(net "SCL")
-	)
-	(segment
-		(start 128.098768 104.241523)
-		(end 128.098768 105.054416)
-		(width 0.254)
-		(layer "F.Cu")
-		(net "SCL")
-	)
-	(via
-		(at 127.501868 105.314643)
-		(size 0.6858)
-		(drill 0.3302)
-		(layers "F.Cu" "B.Cu")
-		(net "SCL")
-	)
-	(segment
-		(start 126.3521 105.01)
-		(end 124.7981 105.01)
-		(width 0.254)
-		(layer "B.Cu")
-		(net "SCL")
-	)
-	(segment
-		(start 126.656743 105.314643)
-		(end 126.3521 105.01)
-		(width 0.254)
-		(layer "B.Cu")
-		(net "SCL")
-	)
-	(segment
-		(start 127.501868 105.314643)
-		(end 126.656743 105.314643)
-		(width 0.254)
-		(layer "B.Cu")
-		(net "SCL")
-	)
-	(segment
 		(start 107.3162 104.232245)
 		(end 107.3162 103.085205)
@@
 	)
 	(segment
-		(start 117.251868 116.16434)
-		(end 117.251868 117.631868)
-		(width 0.254)
-		(layer "F.Cu")
-		(net "Net-(J4-Pin_4)")
-	)
-	(segment
-		(start 117.251868 117.631868)
-		(end 119.350592 119.730592)
-		(width 0.254)
-		(layer "F.Cu")
-		(net "Net-(J4-Pin_4)")
-	)
-	(segment
